File: Hardware/PI_Servo_Shield.sch (EAGLE design)
At the start: 106 parts, among them J1 RASPBERRYPI-40-PIN-GPIO, J19 QWIIC, J20 USB C, J21 Serial, Q1 2N7002PW, Q12 2.5A/30V/105mΩ, Q2 2.5A/30V/105mΩ, Q4 2N7002PW, Q5 2.5A/30V/105mΩ, Q7 2.5A/30V/105mΩ, Q9 2.5A/30V/105mΩ, U1 PCA9685, U2 SN74LVC1G32DCKR, U3 CH340C

Commit message: schematic cleanup and some part positioning
Parts:
- added TP23, TP24, TP25: TEST-POINT3X4, SparkFun-Connectors:TEST-POINT3X4
- D1: device SparkFun-LED:LED-GREEN_HIDDENSILK -> SparkFun-LED:LED-GREEN0603
- D2: value YELLOW -> Yellow; device SparkFun-LED:LED-YELLOW_HIDDENSILK -> SparkFun-LED:LED-YELLOW0603
- JP4: value VIN ISO -> PI ISO
- S1: device SparkFun-Switches:SWITCH-SPDT-PTH-11.6X4.0MM-LOCK -> SparkFun-Switches:SWITCH-SPDT-SMD-RIGHT-ANGLE
Connections:
- new net N$20: JP4.1, Q12.D, R18.2, R19.2
- new net VIN: JP4.2
- net CH340-TXO: now also TP23.1
- net PI-5V: now also TP24.1; no longer JP4.2, Q12.D, R18.2, R19.2
- net PI-RXI: no longer TP21.1
- net RVR-5V: now also TP25.1
- net RVR-TXO: now also TP21.1
- net SERVO: no longer JP4.1
Other:
- note added: "QWIIC"
- note added: "Servo Power Auto-Select"
- note removed: "*Only connect 5V > 5.1 will damage Pi"
- moved on the sheet: C10, C17, C3, C4, C5, C6, C7, C8, D1, D2, F2, J1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
